Commit message: Successful package restructuring

File: neato_simulation/urdf/neato.urdf.xacro (robot description, xacro)
@@ -4,9 +4,9 @@
   be incorporated by other urdf files (e.g. turtlebot).
   See neato_standalone.urdf.xacro for a standalone urdf to be tested with
-      neato_description/launch/view_model.launch
+      neato_simulation/launch/view_model.launch
  -->
 <robot name="neato" xmlns:xacro="http://ros.org/wiki/xacro">
-  <xacro:include filename="$(find neato_description)/urdf/common_properties.urdf.xacro"/>
-  <xacro:include filename="$(find neato_description)/urdf/neato_gazebo.urdf.xacro"/>
+  <xacro:include filename="$(find neato_simulation)/urdf/common_properties.urdf.xacro"/>
+  <xacro:include filename="$(find neato_simulation)/urdf/neato_gazebo.urdf.xacro"/>
   <!-- neato -->
   <xacro:macro name="neato">
@@ -21,5 +21,5 @@
       <visual>
         <geometry>
-          <mesh filename="package://neato_description/meshes/main_body.stl" scale="0.001 0.001 0.001"/>
+          <mesh filename="package://neato_simulation/meshes/main_body.stl" scale="0.001 0.001 0.001"/>
         </geometry>
         <origin xyz="0 0 0" rpy="0 0 0"/>
@@ -55,5 +55,5 @@
       <visual>
         <geometry>
-          <mesh filename="package://neato_description/meshes/wheel.dae"/>
+          <mesh filename="package://neato_simulation/meshes/wheel.dae"/>
         </geometry>
         <origin xyz="0 0 0" rpy="${M_PI/2} 0 0"/>
@@ -82,5 +82,5 @@
       <visual>
         <geometry>
-          <mesh filename="package://neato_description/meshes/wheel.dae"/>
+          <mesh filename="package://neato_simulation/meshes/wheel.dae"/>
         </geometry>
         <origin xyz="0 0 0" rpy="${M_PI/2} 0 0"/>

File: neato_simulation/urdf/neato_standalone.urdf.xacro (robot description, xacro)
@@ -6,5 +6,5 @@
        xmlns:xacro="http://ros.org/wiki/xacro">
   <!-- Defines the neato component tag. -->
-  <xacro:include filename="$(find neato_description)/urdf/neato.urdf.xacro" />
+  <xacro:include filename="$(find neato_simulation)/urdf/neato.urdf.xacro" />
   <xacro:neato/>
 </robot>

Commit message: Fix launch and urdf files for custom package

File: neato_simulation/urdf/neato.urdf.xacro (robot description, xacro)
@@ -24,5 +24,5 @@
         </geometry>
         <origin xyz="0 0 0" rpy="0 0 0"/>
-        <material name="dark_grey"/>
+        <material name="$(arg body_color)"/>
       </visual>
       <collision>

File: neato_simulation/urdf/neato_gazebo.urdf.xacro (robot description, xacro)
@@ -3,5 +3,5 @@
   <xacro:macro name="neato_sim">
     <gazebo reference="base_link">
-      <material>Gazebo/DarkGrey</material>
+      <material>Gazebo/$(arg body_color)</material>
     </gazebo>
     <gazebo reference="wheel_left_link">

Commit message: Complete neato locator implementation

File: neato_simulation/urdf/neato.urdf.xacro (robot description, xacro)
@@ -243,5 +243,5 @@
   <joint name="camera_joint" type="fixed">
     <axis xyz="0 1 0" />
-    <origin xyz="-0.1 0 0.25" rpy="0 0 0"/>
+    <origin xyz="-0 0 0.25" rpy="0 -0.011 0"/>
     <parent link="base_link"/>
     <child link="camera_link"/>
